Commit message: spawns box and atlas in simulator+rviz fixes boston_box mesh resolution increases box mass to 100kg

File: atlas_ros/resource/ground/boston_box.urdf (robot description, URDF)
Before this commit: robot cube, 1 links, 0 joints
Links:
- removed link baseLink
- added link cube_center, mass 100.0; collision box size=1 1 1; visual mesh filename=file://$(find atlas_ros)/resource/ground/boston_box.obj scale=0.5 0.5 0.5

File: robot_model/ground/boston_box.urdf (robot description, URDF)
Before this commit: robot cube, 1 links, 0 joints
Links:
- link baseLink: mass 1.0 -> 100.0
