Commit message: fixes atlas COM dynamics typo? root link of urdf should not have mass, pelvis COM frame is empty, but is not the root of the URDF tree...

File: atlas_ros/resource/atlas/atlas_rel_path.urdf (robot description, URDF)
Before this commit: robot multisense_sl, 34 links, 33 joints
Links:
- link pelvis: mass 9.509 -> 0.001
- link pelvis_com: mass 0.001 -> 9.509

File: robot_model/atlas/atlas.urdf (robot description, URDF)
Before this commit: robot multisense_sl, 34 links, 33 joints
Links:
- link pelvis: mass 9.509 -> 0.001
- link pelvis_com: mass 0.001 -> 9.509
